Commit message: Add rb1 urdf files

File: my_rb1_description/urdf/my_rb1_robot.urdf (robot description, URDF)
Before this commit: robot Rb_1, 7 links, 6 joints
Links:
- link back_caster: geometry collision sphere radius=0.025; collision sphere radius=0.035
- link front_caster: geometry collision sphere radius=0.025; collision sphere radius=0.035

Commit message: Add Pluggins

File: my_rb1_description/urdf/my_rb1_robot.urdf (robot description, URDF)
Before this commit: robot Rb_1, 7 links, 6 joints
Links:
- removed link laserscan
- added link front_laser, mass 0; collision cylinder length=0.020 radius=0.015; visual cylinder length=0.020 radius=0.015
- link left_wheel: geometry collision cylinder length=0.05 radius=0.025; visual cylinder length=0.05 radius=0.025
- link right_wheel: geometry collision cylinder length=0.05 radius=0.025; visual cylinder length=0.05 radius=0.025
Joints:
- joint Laser_joint: child laserscan -> front_laser
- joint joint_baselink_leftwheel: axis 0 -0.2 0 -> 0 0 0
- joint joint_baselink_rightwheel: axis 0 0.2 0 -> 0 0 0

Commit message: Add initial ROS package files

File: my_rb1_description/urdf/my_rb1_robot.urdf (robot description, URDF)
Before this commit: robot Rb_1, 7 links, 6 joints
Links:
- link back_caster: mass 1 -> 0.5
- link front_caster: mass 1 -> 0.5
- link front_laser: mass 0 -> 1
- link left_wheel: geometry collision cylinder length=0.05 radius=0.05; visual cylinder length=0.05 radius=0.05
- link right_wheel: geometry collision cylinder length=0.05 radius=0.05; visual cylinder length=0.05 radius=0.05
Joints:
- joint joint_baselink_leftwheel: axis 0 0 0 -> 0 1 0
- joint joint_baselink_rightwheel: axis 0 0 0 -> 0 1 0

Commit message: Spawn robot

File: my_rb1_description/urdf/my_rb1_robot.urdf (robot description, URDF)
Before this commit: robot Rb_1, 7 links, 6 joints
Links:
- link left_wheel: geometry collision cylinder length=0.05 radius=0.025; visual cylinder length=0.05 radius=0.025
- link right_wheel: geometry collision cylinder length=0.05 radius=0.025; visual cylinder length=0.05 radius=0.025
